File: StickHub.kicad_sch (KiCad schematic)
At the start: 94 parts

Commit message: adding more LEDs
Parts:
- added D26, D27, D28, D29: USB, LED_SMD:Duo_LED_1.6x0.8_Kingbright_APHB1608LZGKSURKC, symbol RobotProtos:LED_DUAL_red_green
- C1: renamed from U; value (none) -> 1uF 10V; footprint (none) -> Capacitor_SMD:1608_C; Spice_Model 100n -> (none); Spice_Netlist_Enabled Y -> (none); Spice_Primitive C -> (none)
- C10, C11, C12, C13, C2, C5, C6, C7, C8, C9: renamed from U; value (none) -> 0.1uF; footprint (none) -> Capacitor_SMD:1608_C; Spice_Model 100n -> (none); Spice_Netlist_Enabled Y -> (none); Spice_Primitive C -> (none)
- C14, C15, C16, C17, C18, C19, C20, C21: renamed from U; value (none) -> 0.1uF 100V; footprint (none) -> Capacitor_SMD:1608_C; Spice_Model 100n -> (none); Spice_Netlist_Enabled Y -> (none); Spice_Primitive C -> (none)
- C22, C23, C24, C25, C26, C27, C29, C30, C31, C32, C33, C34, C35, C36, C37: renamed from U; value (none) -> 22uF 10V; footprint (none) -> Capacitor_SMD:1608_C; Spice_Model 100n -> (none); Spice_Netlist_Enabled Y -> (none); Spice_Primitive C -> (none)
- C28: renamed from U; value (none) -> 15nF; footprint (none) -> Capacitor_SMD:1608_C; Spice_Model 100n -> (none); Spice_Netlist_Enabled Y -> (none); Spice_Primitive C -> (none)
- C3, C4: renamed from U; value (none) -> 10uF 6.3V; footprint (none) -> Capacitor_SMD:1608_C; Spice_Model 100n -> (none); Spice_Netlist_Enabled Y -> (none); Spice_Primitive C -> (none)
- C38: renamed from U; value (none) -> 330uF 10V; footprint (none) -> SH_Capacitors:CP_Elec_6.3x7.7
- D1, D10, D11, D12, D13, D14, D2, D22, D23, D3, D4, D5, D6, D7, D8, D9: renamed from U; value (none) -> TVS; footprint (none) -> Diode_SMD:1006_C
- D15, D16, D17, D18, D19, D20, D21: renamed from U; value (none) -> USB; footprint (none) -> LED_SMD:Duo_LED_1.6x0.8_Kingbright_APHB1608LZGKSURKC
- D24, D25: renamed from U; value (none) -> 5V; footprint (none) -> Diode_SMD:1006_C
- H1: renamed from U; value (none) -> Strap; footprint (none) -> MountingHole:Plain_Hole_3mm
- J1: renamed from U; value (none) -> HOST; footprint (none) -> Connector_USB:USB_A_PCB_traces_small
- J2: renamed from U; value (none) -> USB1; footprint (none) -> Connector_JST:JST_SH_SM04B-SRSS-TB_1x04-1MP_P1.00mm_Horizontal
- J3: renamed from U; value (none) -> USB2; footprint (none) -> Connector_JST:JST_SH_SM04B-SRSS-TB_1x04-1MP_P1.00mm_Horizontal
- J4: renamed from U; value (none) -> USB3; footprint (none) -> Connector_JST:JST_SH_SM04B-SRSS-TB_1x04-1MP_P1.00mm_Horizontal
- J5: renamed from U; value (none) -> USB4; footprint (none) -> Connector_JST:JST_SH_SM04B-SRSS-TB_1x04-1MP_P1.00mm_Horizontal
- J6: renamed from U; value (none) -> USB5; footprint (none) -> Connector_JST:JST_SH_SM04B-SRSS-TB_1x04-1MP_P1.00mm_Horizontal
- J7: renamed from U; value (none) -> USB6; footprint (none) -> Connector_JST:JST_SH_SM04B-SRSS-TB_1x04-1MP_P1.00mm_Horizontal
- J8: renamed from U; value (none) -> USB7; footprint (none) -> Connector_JST:JST_SH_SM04B-SRSS-TB_1x04-1MP_P1.00mm_Horizontal
- J9: renamed from U; value (none) -> EXTGND; footprint (none) -> SH_Solder_Pads:1P-1.5x1.5
- JP1: renamed from U; value (none) -> EXTPWR; footprint (none) -> Connector_PinHeader_2.54mm:PinHeader_1x02_P2.54mm_Vertical
- LOGO1, LOGO2, LOGO3, LOGO4: renamed from U; value (none) -> Logo; footprint (none) -> Logo
- R1: renamed from U; value (none) -> 10k; footprint (none) -> Resistor_SMD:1608_C
- R10, R11, R12, R13, R7, R8, R9: renamed from U; value (none) -> 470; footprint (none) -> Resistor_SMD:1608_C
- R2, R3, R4, R5: renamed from U; value (none) -> 100k; footprint (none) -> Resistor_SMD:1608_C
- R6: renamed from U; value (none) -> 2.7k; footprint (none) -> Resistor_SMD:1608_C
- U1: renamed from U; value (none) -> MaxLinear_XR22417-48; footprint (none) -> Package_QFP:LQFP-48_7x7mm_P0.5mm
- U2: renamed from U; value (none) -> Dialog_SLG5NT1487V; footprint (none) -> Package_DFN_QFN:TDFN-8_1.5x2mm_Fused-Lead_JEDEC_MO-252_W2015D
- Y1: renamed from U; value (none) -> 12MHz 50ppm 16-20pF; footprint (none) -> Crystal:Crystal_4-SMD_2.5x2mm
